File: temp-ref.kicad_pcb (KiCad board)
At the start: 2 copper layers, 37 x 76.5 mm, 51 parts, among them IC1 INA211AIDCKT, IC2 INA211AIDCKT, J1 Conn_01x05_Male, J2 USB_C_Receptacle_USB2.0, J3 Conn_02x05_Odd_Even, Q1 Q_NMOS_GDS, Q2 MMBT3904, Q3 Q_NMOS_GDS, SW1 SW_SPST, SW2 SW_SPST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

Commit message: fixes
Parts:
- removed REF** (x4): MountingHole_3.2mm_M3, MountingHole:MountingHole_3.2mm_M3
Connections:
- U4 pad 49: GND -> (no net)
- U8 pad 2: Net-(U8-Pad2) -> GND
Routing:
- net DALLAS2: track 24.8 -> 26.4 mm
- net DALLAS1: track 20.3 -> 21.7 mm
